File: hardware/MiniTULPAR_KiCAD/MiniTULPAR.kicad_sch (KiCad schematic)
At the start: 0 parts

Commit message: hw: KiCad project and libs file
Other:
- note removed: "Second Acc/Gyro"
Changed lines of the file:
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@@
 	)
 	(rectangle
-		(start 162.814 51.308)
-		(end 180.594 61.468)
+		(start 146.304 65.278)
+		(end 164.084 75.438)
 		(stroke
 			(width 0)
@@
 	)
 	(rectangle
-		(start 147.574 65.913)
-		(end 165.354 76.073)
-		(stroke
-			(width 0)
-			(type solid)
-		)
-		(fill
-			(type color)
-			(color 255 218 94 1)
-		)
-	)
-	(rectangle
 		(start 170.18 78.74)
 		(end 187.96 88.9)
@@
 	(text "CS will be connected to VDD_IO\nSA0 will be connected to GND"
 		(exclude_from_sim no)
-		(at 172.466 48.768 0)
+		(at 155.956 62.738 0)
 		(effects
 			(font
@@
 	(text "I2C"
 		(exclude_from_sim no)
-		(at 161.798 77.978 0)
+		(at 157.226 80.01 0)
 		(effects
 			(font
@@
 		)
 	)
-	(text "Second\nAcc/Gyro"
-		(exclude_from_sim no)
-		(at 156.21 70.485 0)
-		(effects
-			(font
-				(size 1.905 1.905)
-				(thickness 0.381)
-				(bold yes)
-			)
-		)
-	)
 	(text "USB"
 		(exclude_from_sim no)
@@
 	(text "Barometre"
 		(exclude_from_sim no)
-		(at 171.45 55.88 0)
+		(at 154.94 69.85 0)
 		(effects
 			(font
 				(size 1.905 1.905)
 				(thickness 0.2381)
-			)
-		)
-	)
-	(text "SPI"
-		(exclude_from_sim no)
-		(at 154.686 80.518 0)
-		(effects
-			(font
-				(size 0.635 0.635)
-				(thickness 0.254)
-				(bold yes)
 			)
 		)
@@
 	(polyline
 		(pts
-			(xy 155.956 76.2) (xy 155.956 85.09)
-		)
-		(stroke
-			(width 0)
-			(type default)
-		)
-	)
-	(polyline
-		(pts
 			(xy 139.446 129.54) (xy 139.446 132.588)
 		)
@@
 	(polyline
 		(pts
-			(xy 167.894 69.85) (xy 166.116 69.85)
-		)
-		(stroke
-			(width 0)
-			(type default)
-		)
-	)
-	(polyline
-		(pts
 			(xy 129.794 80.264) (xy 124.206 80.264)
 		)
@@
 	(polyline
 		(pts
-			(xy 166.116 78.486) (xy 158.242 78.486)
-		)
-		(stroke
-			(width 0)
-			(type default)
-		)
-	)
-	(polyline
-		(pts
 			(xy 138.684 110.49) (xy 138.684 119.38)
 		)
@@
 	(polyline
 		(pts
-			(xy 158.242 78.486) (xy 158.242 85.09)
+			(xy 158.242 75.438) (xy 158.242 85.09)
 		)
 		(stroke
@@
 	(polyline
 		(pts
-			(xy 166.116 69.85) (xy 166.116 78.486)
-		)
-		(stroke
-			(width 0)
-			(type default)
-		)
-	)
-	(polyline
-		(pts
 			(xy 135.89 76.2) (xy 135.89 85.09)
-		)
-		(stroke
-			(width 0)
-			(type default)
-		)
-	)
-	(polyline
-		(pts
-			(xy 167.894 61.468) (xy 167.894 69.85)
 		)
 		(stroke
@@
 	)
 	(group ""
-		(members "67d1440b-db7c-4644-914e-c71772d6c36f" "f18c9359-74fb-476c-b9b0-ce9f5d1d6e23")
-	)
-	(group ""
